Commit message: Some changes for the tests

File: birmingham_cell_description/urdf/panda_pybullet.urdf (robot description, URDF)
Before this commit: robot panda, 19 links, 18 joints
Links:
- link panda_hand: geometry collision mesh filename=/home/battery/michele_projects/personal_ws/src/birmingham_c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; visual mesh filename=/home/battery/michele_projects/personal_ws/src/birmingham_c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
- link panda_leftfinger: geometry collision mesh filename=/home/battery/michele_projects/personal_ws/src/birmingham_c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; visual mesh filename=/home/battery/michele_projects/personal_ws/src/birmingham_c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
- link panda_link0: geometry collision mesh filename=/home/battery/michele_projects/personal_ws/src/birmingham_c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; visual mesh filename=/home/battery/michele_projects/personal_ws/src/birmingham_c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
- link panda_link1: geometry collision mesh filename=/home/battery/michele_projects/personal_ws/src/birmingham_c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; visual mesh filename=/home/battery/michele_projects/personal_ws/src/birmingham_c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
- link panda_link2: geometry collision mesh filename=/home/battery/michele_projects/personal_ws/src/birmingham_c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; visual mesh filename=/home/battery/michele_projects/personal_ws/src/birmingham_c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
- link panda_link3: geometry collision mesh filename=/home/battery/michele_projects/personal_ws/src/birmingham_c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; visual mesh filename=/home/battery/michele_projects/personal_ws/src/birmingham_c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
- link panda_link4: geometry collision mesh filename=/home/battery/michele_projects/personal_ws/src/birmingham_c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; visual mesh filename=/home/battery/michele_projects/personal_ws/src/birmingham_c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
- link panda_link5: geometry collision mesh filename=/home/battery/michele_projects/personal_ws/src/birmingham_c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; visual mesh filename=/home/battery/michele_projects/personal_ws/src/birmingham_c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
- link panda_link6: geometry collision mesh filename=/home/battery/michele_projects/personal_ws/src/birmingham_c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; visual mesh filename=/home/battery/michele_projects/personal_ws/src/birmingham_c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
- link panda_link7: geometry collision mesh filename=/home/battery/michele_projects/personal_ws/src/birmingham_c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; visual mesh filename=/home/battery/michele_projects/personal_ws/src/birmingham_c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
- link panda_rightfinger: geometry collision mesh filename=/home/battery/michele_projects/personal_ws/src/birmingham_c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; visual mesh filename=/home/battery/michele_projects/personal_ws/src/birmingham_c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

Commit message: Fix error with params to not change

File: birmingham_cell_description/urdf/panda_pybullet.urdf (robot description, URDF)
Before this commit: robot panda, 19 links, 18 joints
Links:
- link panda_hand: geometry collision mesh filename=/home/gauss/projects/personal_ws/src/birmingham_cell/birmin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; visual mesh filename=/home/gauss/projects/personal_ws/src/birmingham_cell/birmin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
- link panda_leftfinger: geometry collision mesh filename=/home/gauss/projects/personal_ws/src/birmingham_cell/birmin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; visual mesh filename=/home/gauss/projects/personal_ws/src/birmingham_cell/birmin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
- link panda_link0: geometry collision mesh filename=/home/gauss/projects/personal_ws/src/birmingham_cell/birmin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; visual mesh filename=/home/gauss/projects/personal_ws/src/birmingham_cell/birmin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
- link panda_link1: geometry collision mesh filename=/home/gauss/projects/personal_ws/src/birmingham_cell/birmin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; visual mesh filename=/home/gauss/projects/personal_ws/src/birmingham_cell/birmin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
- link panda_link2: geometry collision mesh filename=/home/gauss/projects/personal_ws/src/birmingham_cell/birmin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; visual mesh filename=/home/gauss/projects/personal_ws/src/birmingham_cell/birmin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
- link panda_link3: geometry collision mesh filename=/home/gauss/projects/personal_ws/src/birmingham_cell/birmin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; visual mesh filename=/home/gauss/projects/personal_ws/src/birmingham_cell/birmin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
- link panda_link4: geometry collision mesh filename=/home/gauss/projects/personal_ws/src/birmingham_cell/birmin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; visual mesh filename=/home/gauss/projects/personal_ws/src/birmingham_cell/birmin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
- link panda_link5: geometry collision mesh filename=/home/gauss/projects/personal_ws/src/birmingham_cell/birmin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; visual mesh filename=/home/gauss/projects/personal_ws/src/birmingham_cell/birmin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
- link panda_link6: geometry collision mesh filename=/home/gauss/projects/personal_ws/src/birmingham_cell/birmin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; visual mesh filename=/home/gauss/projects/personal_ws/src/birmingham_cell/birmin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
- link panda_link7: geometry collision mesh filename=/home/gauss/projects/personal_ws/src/birmingham_cell/birmin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; visual mesh filename=/home/gauss/projects/personal_ws/src/birmingham_cell/birmin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
- link panda_rightfinger: geometry collision mesh filename=/home/gauss/projects/personal_ws/src/birmingham_cell/birmin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; visual mesh filename=/home/gauss/projects/personal_ws/src/birmingham_cell/birmin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
