Commit message: General model tested on simulation environment

File: birmingham_cell_description/urdf/box.urdf (robot description, URDF)
Before this commit: robot box_model, 1 links, 0 joints
Links:
- link box: geometry collision box size=0.04 0.03 0.07; visual box size=0.04 0.03 0.07

File: birmingham_cell_description/urdf/cylinder.urdf (robot description, URDF)
Before this commit: robot cylinder_model, 1 links, 0 joints
Links:
- link cylinder: geometry collision cylinder length=0.04 radius=0.03; visual cylinder length=0.04 radius=0.03

File: birmingham_cell_description/urdf/sphere.urdf (robot description, URDF)
Before this commit: robot sphere_model, 1 links, 0 joints
Links:
- link sphere: geometry collision sphere radius=0.03; visual sphere radius=0.03
