Commit message: Box and cylinder hole added

File: birmingham_cell_description/urdf/box_hole.urdf (robot description, URDF)
Before this commit: robot box_model, 1 links, 0 joints
Links:
- removed link box
- added link box_hole, mass 0.390; collision mesh filename=package://birmingham_cell_description/meshes/Box_hole.STL scale=0.04 0.04 0.06; visual mesh filename=package://birmingham_cell_description/meshes/Box_hole.STL scale=0.04 0.04 0.06

File: birmingham_cell_description/urdf/cylinder.urdf (robot description, URDF)
Before this commit: robot cylinder_model, 1 links, 0 joints
Links:
- link cylinder: geometry collision cylinder length=0.1 radius=0.02; visual cylinder length=0.1 radius=0.02

File: birmingham_cell_description/urdf/cylinder_hole.urdf (robot description, URDF)
Before this commit: robot box_model, 1 links, 0 joints
Links:
- removed link box
- added link cylinder_hole, mass 0.390; collision mesh filename=package://birmingham_cell_description/meshes/Cylinder_hole.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 scale=0.045 0.045 0.06; visual mesh filename=package://birmingham_cell_description/meshes/Cylinder_hole.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 scale=0.045 0.045 0.06

File: birmingham_cell_description/urdf/hand.xacro (robot description, xacro)
@@ -53,5 +53,6 @@
         </material>
       </visual>
-      <collision>
+      <!-- <collision> -->
+      <collision concave="yes">
         <geometry>
           <mesh filename="package://birmingham_cell_description/meshes/leftfinger_collision.STL"/>
@@ -81,5 +82,6 @@
         </material>
       </visual>
-      <collision>
+      <!-- <collision> -->
+      <collision concave="yes">
         <geometry>
           <mesh filename="package://birmingham_cell_description/meshes/rightfinger_collision.STL"/>
