Commit message: Change total_reward

File: birmingham_cell_description/urdf/hand.xacro (robot description, xacro)
@@ -93,5 +93,5 @@
       <axis xyz="0 1 0"/>
       <limit effort="20" lower="-0.001" upper="0.04" velocity="0.3"/>
-      <mimic joint="${ns}_left_joint_circle" multiplier="0.08" offset="0" />
+      <mimic joint="${ns}_left_joint_circle" multiplier="0.04" offset="0" />
     </joint>
     <joint name="${ns}_finger_joint2" type="prismatic">

File: birmingham_cell_description/urdf/panda_pybullet.urdf (robot description, URDF)
Before this commit: robot panda, 19 links, 18 joints
Links:
- link panda_hand: geometry collision mesh filename=/home/gauss/projects/personal_ws/src/birmingham_cell/birmin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; visual mesh filename=/home/gauss/projects/personal_ws/src/birmingham_cell/birmin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
- link panda_leftfinger: geometry collision mesh filename=/home/gauss/projects/personal_ws/src/birmingham_cell/birmin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; visual mesh filename=/home/gauss/projects/personal_ws/src/birmingham_cell/birmin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
- link panda_link0: geometry collision mesh filename=/home/gauss/projects/personal_ws/src/birmingham_cell/birmin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; visual mesh filename=/home/gauss/projects/personal_ws/src/birmingham_cell/birmin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
- link panda_link1: geometry collision mesh filename=/home/gauss/projects/personal_ws/src/birmingham_cell/birmin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; visual mesh filename=/home/gauss/projects/personal_ws/src/birmingham_cell/birmin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
- link panda_link2: geometry collision mesh filename=/home/gauss/projects/personal_ws/src/birmingham_cell/birmin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; visual mesh filename=/home/gauss/projects/personal_ws/src/birmingham_cell/birmin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
- link panda_link3: geometry collision mesh filename=/home/gauss/projects/personal_ws/src/birmingham_cell/birmin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; visual mesh filename=/home/gauss/projects/personal_ws/src/birmingham_cell/birmin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
- link panda_link4: geometry collision mesh filename=/home/gauss/projects/personal_ws/src/birmingham_cell/birmin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; visual mesh filename=/home/gauss/projects/personal_ws/src/birmingham_cell/birmin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
- link panda_link5: geometry collision mesh filename=/home/gauss/projects/personal_ws/src/birmingham_cell/birmin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; visual mesh filename=/home/gauss/projects/personal_ws/src/birmingham_cell/birmin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
- link panda_link6: geometry collision mesh filename=/home/gauss/projects/personal_ws/src/birmingham_cell/birmin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; visual mesh filename=/home/gauss/projects/personal_ws/src/birmingham_cell/birmin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
- link panda_link7: geometry collision mesh filename=/home/gauss/projects/personal_ws/src/birmingham_cell/birmin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; visual mesh filename=/home/gauss/projects/personal_ws/src/birmingham_cell/birmin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
- link panda_rightfinger: geometry collision mesh filename=/home/gauss/projects/personal_ws/src/birmingham_cell/birmin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; visual mesh filename=/home/gauss/projects/personal_ws/src/birmingham_cell/birmin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
Joints:
- joint panda_finger_joint1: mimic joint=panda_left_joint_circle multiplier=0.08 offset=0 -> joint=panda_left_joint_circle multiplier=0.04 offset=0

Commit message: realistic_fake_env added

File: birmingham_cell_description/urdf/hand.xacro (robot description, xacro)
@@ -93,5 +93,5 @@
       <axis xyz="0 1 0"/>
       <limit effort="20" lower="-0.001" upper="0.04" velocity="0.3"/>
-      <mimic joint="${ns}_left_joint_circle" multiplier="0.04" offset="0" />
+      <!-- <mimic joint="${ns}_left_joint_circle" multiplier="0.07" offset="0" /> -->
     </joint>
     <joint name="${ns}_finger_joint2" type="prismatic">

File: birmingham_cell_description/urdf/panda_pybullet.urdf (robot description, URDF)
Before this commit: robot panda, 19 links, 18 joints
Joints:
- joint panda_finger_joint1: mimic joint=panda_left_joint_circle multiplier=0.04 offset=0 -> (none)

Commit message: ready to collect data

File: birmingham_cell_description/urdf/hand.xacro (robot description, xacro)
@@ -31,5 +31,5 @@
       </collision>
     </link>
-    <link name="${ns}_leftfinger">
+    <link name="${ns}_leftfinger" concave="yes">
       <contact>
         <friction_anchor/>
@@ -60,5 +60,5 @@
       </collision>
     </link>
-    <link name="${ns}_rightfinger">
+    <link name="${ns}_rightfinger" concave="yes">
       <contact>
         <friction_anchor/>

Commit message: Ready to collect complex task data

File: birmingham_cell_description/urdf/hand.xacro (robot description, xacro)
@@ -31,5 +31,5 @@
       </collision>
     </link>
-    <link name="${ns}_leftfinger" concave="yes">
+    <link name="${ns}_leftfinger">
       <contact>
         <friction_anchor/>
@@ -54,5 +54,5 @@
       </visual>
       <!-- <collision> -->
-      <collision concave="yes">
+      <collision>
         <geometry>
           <mesh filename="package://birmingham_cell_description/meshes/leftfinger_collision.STL"/>
@@ -60,5 +60,5 @@
       </collision>
     </link>
-    <link name="${ns}_rightfinger" concave="yes">
+    <link name="${ns}_rightfinger">
       <contact>
         <friction_anchor/>
@@ -83,5 +83,5 @@
       </visual>
       <!-- <collision> -->
-      <collision concave="yes">
+      <collision>
         <geometry>
           <mesh filename="package://birmingham_cell_description/meshes/rightfinger_collision.STL"/>
